File: ECAD/Iridium.kicad_sch (KiCad schematic)
At the start: 21 parts

Commit message: add footprints and update iridium section
Parts:
- AE1: renamed from AE?; footprint (none) -> Connector_Coaxial:SMA_Amphenol_901-143_Horizontal
- R2: renamed from R?; value 10m -> 4m; footprint (none) -> Resistor_SMD:R_1206_3216Metric
- U6: renamed from U?; value INA138 -> INA180A3
- gave numbers to parts that had none: 18
Connections:
- net +BATT renamed SW1
