File: iridium-bus/piridium-bus.kicad_sch (KiCad schematic)
At the start: 2 parts

Commit message: sch milestone
Parts:
- added A?: 9602N, symbol piridium-bus:9602N
- added BT?: CR2032, symbol Device:Battery_Cell
- added C? (x3): 0.1uF, symbol Device:C
- added C? (x4): 22uF, symbol Device:C
- added C? (x3): 10uF, symbol Device:C
- added C? (x3): 1uF, symbol Device:C
- added D?: LED, symbol Device:LED
- added H? (x4): M3, symbol Mechanical:MountingHole_Pad
- added J?: MODEM UART, symbol Connector:Conn_01x06_Male
- added J?: ANT, symbol Connector:Conn_Coaxial
- added JP?: WDT_EN, symbol Jumper:Jumper_2_Open
- added L? (x2): 4.7uH, symbol Device:L
- added R? (x2): 22.1K, symbol Device:R
- added R? (x2): 100K, symbol Device:R
- added R? (x2): 10K, symbol Device:R
- added R? (x2): 124K, symbol Device:R
- added TP? (x2): GND, symbol Connector:TestPoint
- added TP?: 5V, symbol Connector:TestPoint
- added TP?: 5VP, symbol Connector:TestPoint
- added U1: MAX6369, Package_TO_SOT_SMD:SOT-23-8, symbol Power_Supervisor:MAX6369
- added U2: TPS54394RSAR, Package_DFN_QFN:Texas_S-PVQFN-N16_EP2.7x2.7mm_ThermalVias, symbol iridium-bus:TPS54394RSAR
- added U3: DS3232M, Package_SO:SOIC-8_3.9x4.9mm_P1.27mm, symbol Timer_RTC:DS3232M
- added U?: LM1117-3.3, symbol Regulator_Linear:LM1117-3.3
- A1: renamed from A?; footprint (none) -> piridium-bus:Raspberry Pi Zero
- A2: renamed from A?; footprint (none) -> piridium-bus:BNO055
Connections:
- net +3.3V: now reaches A1.1 (3V3)
- net +3.3V: now also A1.17 (3V3), A2.1 (VIN), C?.2, U3.2 (VCC)
- net UART_RX: now reaches A1.10 (15(RxD))
- net UART_RX: now also A?.7 (DF_S_RX), J?.2 (Pin_2)
- net GND: now reaches A1.14 (GND)
- net GND: now also A1.20 (GND), A1.25 (GND), A1.30 (GND), A1.34 (GND), A1.39 (GND), A1.6 (GND), A1.9 (GND), A2.3 (GND), A?.14 (DF_DTR), A?.15 (SIG_GND), A?.18 (SIG_GND), A?.22 (RF_GND), A?.3 (EXT_GND), A?.4 (EXT_GND), A?.8 (SIG_GND), BT?.2 (-), C?.1, C?.2, C?.2, C?.2, C?.2, C?.2, C?.2, C?.2, C?.2, C?.2, C?.2, D?.1 (K), H?.1, H?.1, H?.1, H?.1, J?.2 (Ext), J?.6 (Pin_6), R?.2, R?.2, R?.2, TP?.1, TP?.1, U1.2 (GND), U2.10 (GND), U2.15 (PGND2), U2.17 (PADGND), U2.6 (PGND1), U3.5 (GND), U?.1 (GND)
- net SPI_MOSI: now reaches A1.19 (10(MOSI))
- net +5V: now reaches A1.2 (5V)
- net +5V: now also A1.4 (5V), C?.1, C?.1, L?.1, R?.1, R?.1, TP?.1
- net SPI_MISO: now reaches A1.21 (9(MISO))
- net SPI_SCK: now reaches A1.23 (11(SCK))
- net SPI_CE0: now reaches A1.24 (8(CE0))
- net SPI_CE1: now reaches A1.26 (7(CE1))
- net I2C_SDA: now reaches A1.3 (2(SDA1))
- net I2C_SDA: now also A2.4 (SDA), U3.7 (SDA)
- net NET_AVAIL: now reaches A1.32 (12(PWM0))
- net NET_AVAIL: now also A?.19 (NET_AVAIL)
- net RING_INDICATOR: now reaches A1.36 (16)
- net RING_INDICATOR: now also A?.12 (DF_RI)
- net MODEM_ON_OFF: now reaches A1.38 (20)
- net MODEM_ON_OFF: now also A?.5 (ON/OFF), R?.2
- net HANDSHAKE: now reaches A1.40 (21)
- net HANDSHAKE: now also R?.1, U1.1 (WDI)
- net I2C_SCL: now reaches A1.5 (3(SCL1))
- net I2C_SCL: now also A2.5 (SCL), U3.8 (SCL)
- net UART_TX: now reaches A1.8 (14(TxD))
- net UART_TX: now also A?.6 (DF_S_TX), J?.3 (Pin_3)
- new net: C?.1, U2.4 (VBST1)
- new net: C?.2, L?.2, U2.5 (SW1)
- new net: R?.1, R?.2, U2.12 (VFB2)
- new net: C?.1, R?.1, U1.4 (SET0), U1.5 (SET1), U1.6 (SET2), U1.8 (VCC), U?.2 (VO)
- new net: JP?.1 (A), U1.7 (~{WDO})
- new net: R?.1, R?.2, U2.9 (VFB1)
- new net: BT?.1 (+), C?.1, U3.6 (VBAT)
- new net: C?.1, U2.1 (VBST2)
- new net: C?.2, L?.1, U2.16 (SW2)
- new net: A?.20 (SUPPLY_OUT), R?.1
- new net: D?.2 (A), R?.2
- new net: A?.21 (RF_ANT), J?.1 (In)
- new net: C?.1, U2.11 (VREG5)
- new net +5VP: A?.1 (EXT_PWR), A?.2 (EXT_PWR), C?.1, C?.1, L?.2, R?.1, TP?.1
- new net +BATT: C?.1, C?.1, C?.1, U2.2 (VIN2), U2.3 (VIN1), U?.3 (VI)
- new net EN: JP?.2 (B), R?.2, U2.14 (EN2), U2.7 (EN1)
- new net UART_CTS: A?.11 (DF_CTS), J?.5 (Pin_5)
- new net UART_RTS: A?.13 (DF_RTS), J?.1 (Pin_1)
- no-connect marks 0 -> 15
Other:
- note added: "All logic is 3.3V logic level, but is 5V tolerant TX and RX are from master device (TX is input to the 9602, RX is output from the 9602)"
- note added: "Dual 5V Regulator"
- note added: "IMU Breakout Board"
- note added: "Iridium 9602N Modem"
- note added: "Isolated 5V Rail for Modem"
- note added: "Main 5V Rail"
- note added: "Raspi Zero Flight Computer"
- note added: "Real Time Clock & Battery Backup"
- note added: "Resets power if a signal is not received every 60 seconds"
- note added: "Supply indicator LED"
- note added: "TODO: Tristate buffer the 9602 Modem Add power input connector and EPS telemetry? Add power and data output connector"
- note added: "This thing is really picky about power: 5V, <100mVpp 0-50KHz, <10mVpp 1MHz, <5mVpp 5Mhz Transients spikes during xmit from 40mA (idle) to 1.5A (xmit) for 8.3ms Cannot droop below 4.8V during this time OCP required, and in-rush current limit to 4A"
- note added: "Watchdog Timer"
- moved on the sheet: A1, A2
