File: piridium-bus/piridium-bus.kicad_sch (KiCad schematic)
At the start: 52 parts, among them J1 EPS, J2 MODEM UART, J3 ANT, J4 PAYLOAD, Q1 2N7002, Q2 DMP3015LSSQ, U1 LM1117-3.3, U2 TPS54394RSAR, U3 MAX6369, U4 74LS126, U5 DS3232M

Commit message: some work on routing
Parts:
- C6, C7: footprint Capacitor_SMD:C_0805_2012Metric -> Capacitor_SMD:C_0603_1608Metric
- renumbered H1 to MH1, H2 to MH2, H3 to MH3, H4 to MH4
Changed lines of the file:
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@@
       (effects (font (size 1.27 1.27)) (justify left))
     )
-    (property "Footprint" "Capacitor_SMD:C_0805_2012Metric" (id 2) (at 48.5648 114.3 0)
+    (property "Footprint" "Capacitor_SMD:C_0603_1608Metric" (id 2) (at 48.5648 114.3 0)
       (effects (font (size 1.27 1.27)) hide)
     )
@@
   (symbol (lib_id "Mechanical:MountingHole_Pad") (at 261.62 53.34 0) (unit 1)
     (in_bom yes) (on_board yes) (fields_autoplaced)
-    (property "Reference" "H4" (id 0) (at 264.16 50.7999 0)
+    (property "Reference" "MH4" (id 0) (at 264.16 50.7999 0)
       (effects (font (size 1.27 1.27)) (justify left))
     )
@@
   (symbol (lib_id "Mechanical:MountingHole_Pad") (at 234.95 53.34 0) (unit 1)
     (in_bom yes) (on_board yes) (fields_autoplaced)
-    (property "Reference" "H1" (id 0) (at 237.49 50.7999 0)
+    (property "Reference" "MH1" (id 0) (at 237.49 50.7999 0)
       (effects (font (size 1.27 1.27)) (justify left))
     )
@@
   (symbol (lib_id "Mechanical:MountingHole_Pad") (at 243.84 53.34 0) (unit 1)
     (in_bom yes) (on_board yes) (fields_autoplaced)
-    (property "Reference" "H2" (id 0) (at 246.38 50.7999 0)
+    (property "Reference" "MH2" (id 0) (at 246.38 50.7999 0)
       (effects (font (size 1.27 1.27)) (justify left))
     )
@@
       (effects (font (size 1.27 1.27)) (justify left))
     )
-    (property "Footprint" "Capacitor_SMD:C_0805_2012Metric" (id 2) (at 73.3552 114.3 0)
+    (property "Footprint" "Capacitor_SMD:C_0603_1608Metric" (id 2) (at 73.3552 114.3 0)
       (effects (font (size 1.27 1.27)) hide)
     )
@@
   (symbol (lib_id "Mechanical:MountingHole_Pad") (at 252.73 53.34 0) (unit 1)
     (in_bom yes) (on_board yes) (fields_autoplaced)
-    (property "Reference" "H3" (id 0) (at 255.27 50.7999 0)
+    (property "Reference" "MH3" (id 0) (at 255.27 50.7999 0)
       (effects (font (size 1.27 1.27)) (justify left))
     )
@@
     )
     (path "/0a6fd6c8-d7db-4d3e-b044-c1ca2429107f"
-      (reference "C6") (unit 1) (value "0.1uF") (footprint "Capacitor_SMD:C_0805_2012Metric")
+      (reference "C6") (unit 1) (value "0.1uF") (footprint "Capacitor_SMD:C_0603_1608Metric")
     )
     (path "/55c0baef-5360-4ac7-886a-d6cdbe2f49a6"
-      (reference "C7") (unit 1) (value "0.1uF") (footprint "Capacitor_SMD:C_0805_2012Metric")
+      (reference "C7") (unit 1) (value "0.1uF") (footprint "Capacitor_SMD:C_0603_1608Metric")
     )
     (path "/801272d8-944f-4d2f-b54d-b52fcaccc798"
@@
       (reference "D1") (unit 1) (value "LED") (footprint "LED_SMD:LED_0805_2012Metric")
     )
-    (path "/38c8b968-ed8b-48c3-8f10-00c9302564af"
-      (reference "H1") (unit 1) (value "M3") (footprint "MountingHole:MountingHole_3.2mm_M3_DIN965_Pad")
-    )
-    (path "/521323a6-d8a6-4440-944c-03c95480786b"
-      (reference "H2") (unit 1) (value "M3") (footprint "MountingHole:MountingHole_3.2mm_M3_DIN965_Pad")
-    )
-    (path "/9958619c-b644-4318-a651-1582659c7391"
-      (reference "H3") (unit 1) (value "M3") (footprint "MountingHole:MountingHole_3.2mm_M3_DIN965_Pad")
-    )
-    (path "/225cc74f-319d-4c48-80fd-7620a86ed3c6"
-      (reference "H4") (unit 1) (value "M3") (footprint "MountingHole:MountingHole_3.2mm_M3_DIN965_Pad")
-    )
     (path "/321ea199-1ef7-40a0-ade9-c079749b846a"
       (reference "J1") (unit 1) (value "EPS") (footprint "Connector_Molex:Molex_Nano-Fit_105313-xx04_1x04_P2.50mm_Horizontal")
@@
       (reference "L2") (unit 1) (value "4.7uH") (footprint "Inductor_SMD:L_Abracon_ASPI-0630LR")
     )
+    (path "/38c8b968-ed8b-48c3-8f10-00c9302564af"
+      (reference "MH1") (unit 1) (value "M3") (footprint "MountingHole:MountingHole_3.2mm_M3_DIN965_Pad")
+    )
+    (path "/521323a6-d8a6-4440-944c-03c95480786b"
+      (reference "MH2") (unit 1) (value "M3") (footprint "MountingHole:MountingHole_3.2mm_M3_DIN965_Pad")
+    )
+    (path "/9958619c-b644-4318-a651-1582659c7391"
+      (reference "MH3") (unit 1) (value "M3") (footprint "MountingHole:MountingHole_3.2mm_M3_DIN965_Pad")
+    )
+    (path "/225cc74f-319d-4c48-80fd-7620a86ed3c6"
+      (reference "MH4") (unit 1) (value "M3") (footprint "MountingHole:MountingHole_3.2mm_M3_DIN965_Pad")
+    )
     (path "/2f03028b-6b92-4188-b01e-2bc64a9982ab"

Commit message: routing work on bus
Parts:
- added R11: 33K, Resistor_SMD:R_1206_3216Metric, symbol Device:R
- R10, R3, R4, R7, R8: footprint Resistor_SMD:R_0805_2012Metric -> Resistor_SMD:R_1206_3216Metric
- R12: renamed from R11; footprint Resistor_SMD:R_0805_2012Metric -> Resistor_SMD:R_1206_3216Metric
- R9: value 10K -> 22K; footprint Resistor_SMD:R_0805_2012Metric -> Resistor_SMD:R_1206_3216Metric
Connections:
- net GND: now also R11.1
- net S_MODEM_ON_OFF: now also R11.2
Changed lines of the file:
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@@
   (junction (at 20.32 129.54) (diameter 0) (color 0 0 0 0)
+  )
+  (junction (at 240.03 99.06) (diameter 0) (color 0 0 0 0)
   )
   (junction (at 99.06 57.15) (diameter 0) (color 0 0 0 0)
@@
     (stroke (width 0) (type default) (color 0 0 0 0))
   )
-  (wire (pts (xy 233.68 99.06) (xy 242.57 99.06))
+  (wire (pts (xy 233.68 99.06) (xy 240.03 99.06))
     (stroke (width 0) (type default) (color 0 0 0 0))
   )
@@
     (stroke (width 0) (type default) (color 0 0 0 0))
   )
+  (wire (pts (xy 240.03 88.9) (xy 245.11 88.9))
+    (stroke (width 0) (type default) (color 0 0 0 0))
+  )
   (wire (pts (xy 99.06 31.75) (xy 99.06 36.83))
     (stroke (width 0) (type default) (color 0 0 0 0))
@@
     (stroke (width 0) (type default) (color 0 0 0 0))
   )
+  (wire (pts (xy 240.03 99.06) (xy 242.57 99.06))
+    (stroke (width 0) (type default) (color 0 0 0 0))
+  )
   (wire (pts (xy 234.95 35.56) (xy 234.95 38.1))
     (stroke (width 0) (type default) (color 0 0 0 0))
@@
   )
   (wire (pts (xy 87.63 114.3) (xy 92.71 114.3))
+    (stroke (width 0) (type default) (color 0 0 0 0))
+  )
+  (wire (pts (xy 240.03 91.44) (xy 240.03 88.9))
     (stroke (width 0) (type default) (color 0 0 0 0))
   )
@@
     )
     (property "Value" "100K" (id 1) (at 45.72 46.99 90))
-    (property "Footprint" "Resistor_SMD:R_0805_2012Metric" (id 2) (at 43.942 46.99 90)
+    (property "Footprint" "Resistor_SMD:R_1206_3216Metric" (id 2) (at 43.942 46.99 90)
       (effects (font (size 1.27 1.27)) hide)
     )
@@
     (pin "1")
   )
+  (symbol (lib_id "power:GND") (at 245.11 88.9 0) (unit 1)
+    (in_bom yes) (on_board yes)
+    (property "Reference" "#PWR031" (id 0) (at 245.11 95.25 0)
+      (effects (font (size 1.27 1.27)) hide)
+    )
+    (property "Value" "GND" (id 1) (at 245.11 92.71 0))
+    (property "Footprint" "" (id 2) (at 245.11 88.9 0)
+      (effects (font (size 1.27 1.27)) hide)
+    )
+    (property "Datasheet" "" (id 3) (at 245.11 88.9 0)
+      (effects (font (size 1.27 1.27)) hide)
+    )
+    (pin "1")
+  )
   (symbol (lib_id "power:GND") (at 25.4 99.06 0) (unit 1)
     (in_bom yes) (on_board yes)
@@
     (pin "2")
   )
+  (symbol (lib_id "Device:R") (at 240.03 95.25 0) (unit 1)
+    (in_bom yes) (on_board yes)
+    (property "Reference" "R11" (id 0) (at 241.3 95.25 0)
+      (effects (font (size 1.27 1.27)) (justify left))
+    )
+    (property "Value" "33K" (id 1) (at 240.03 95.25 90))
+    (property "Footprint" "Resistor_SMD:R_1206_3216Metric" (id 2) (at 238.252 95.25 90)
+      (effects (font (size 1.27 1.27)) hide)
+    )
+    (property "Datasheet" "~" (id 3) (at 240.03 95.25 0)
+      (effects (font (size 1.27 1.27)) hide)
+    )
+    (pin "1")
+    (pin "2")
+  )
   (symbol (lib_id "power:+BATT") (at 247.65 17.78 0) (unit 1)
     (in_bom yes) (on_board yes)
-    (property "Reference" "#PWR031" (id 0) (at 247.65 21.59 0)
+    (property "Reference" "#PWR032" (id 0) (at 247.65 21.59 0)
       (effects (font (size 1.27 1.27)) hide)
     )
@@
     )
     (property "Value" "100K" (id 1) (at 86.36 39.37 90))
-    (property "Footprint" "Resistor_SMD:R_0805_2012Metric" (id 2) (at 84.582 39.37 90)
+    (property "Footprint" "Resistor_SMD:R_1206_3216Metric" (id 2) (at 84.582 39.37 90)
       (effects (font (size 1.27 1.27)) hide)
     )
@@
     (property "Reference" "R7" (id 0) (at 223.52 27.94 90))
     (property "Value" "100R" (id 1) (at 223.52 30.48 90))
-    (property "Footprint" "Resistor_SMD:R_0805_2012Metric" (id 2) (at 223.52 32.258 90)
+    (property "Footprint" "Resistor_SMD:R_1206_3216Metric" (id 2) (at 223.52 32.258 90)
       (effects (font (size 1.27 1.27)) hide)
     )
@@
   (symbol (lib_id "Device:R") (at 247.65 101.6 90) (unit 1)
     (in_bom yes) (on_board yes)
-    (property "Reference" "R11" (id 0) (at 247.65 104.14 90))
+    (property "Reference" "R12" (id 0) (at 247.65 104.14 90))
     (property "Value" "10K" (id 1) (at 247.65 101.6 90))
-    (property "Footprint" "Resistor_SMD:R_0805_2012Metric" (id 2) (at 247.65 103.378 90)
+    (property "Footprint" "Resistor_SMD:R_1206_3216Metric" (id 2) (at 247.65 103.378 90)
       (effects (font (size 1.27 1.27)) hide)
     )
@@
   (symbol (lib_id "power:GND") (at 265.43 40.64 0) (unit 1)
     (in_bom yes) (on_board yes)
-    (property "Reference" "#PWR034" (id 0) (at 265.43 46.99 0)
+    (property "Reference" "#PWR035" (id 0) (at 265.43 46.99 0)
       (effects (font (size 1.27 1.27)) hide)
     )
@@
   (symbol (lib_id "power:GND") (at 278.13 40.64 0) (unit 1)
     (in_bom yes) (on_board yes)
-    (property "Reference" "#PWR035" (id 0) (at 278.13 46.99 0)
+    (property "Reference" "#PWR036" (id 0) (at 278.13 46.99 0)
       (effects (font (size 1.27 1.27)) hide)
     )
@@
       (effects (font (size 1.27 1.27)) (justify left))
     )
-    (property "Value" "10K" (id 1) (at 233.68 95.25 90))
-    (property "Footprint" "Resistor_SMD:R_0805_2012Metric" (id 2) (at 231.902 95.25 90)
+    (property "Value" "22K" (id 1) (at 233.68 95.25 90))
+    (property "Footprint" "Resistor_SMD:R_1206_3216Metric" (id 2) (at 231.902 95.25 90)
       (effects (font (size 1.27 1.27)) hide)
     )
@@
     )
     (property "Value" "10K" (id 1) (at 227.33 34.29 90))
-    (property "Footprint" "Resistor_SMD:R_0805_2012Metric" (id 2) (at 229.108 34.29 90)
+    (property "Footprint" "Resistor_SMD:R_1206_3216Metric" (id 2) (at 229.108 34.29 90)
       (effects (font (size 1.27 1.27)) hide)
     )
@@
     )
     (property "Value" "10K" (id 1) (at 234.95 21.59 90))
-    (property "Footprint" "Resistor_SMD:R_0805_2012Metric" (id 2) (at 236.728 21.59 90)
+    (property "Footprint" "Resistor_SMD:R_1206_3216Metric" (id 2) (at 236.728 21.59 90)
       (effects (font (size 1.27 1.27)) hide)
     )
@@
   (symbol (lib_id "power:GND") (at 251.46 109.22 0) (unit 1)
     (in_bom yes) (on_board yes) (fields_autoplaced)
-    (property "Reference" "#PWR033" (id 0) (at 251.46 115.57 0)
+    (property "Reference" "#PWR034" (id 0) (at 251.46 115.57 0)
       (effects (font (size 1.27 1.27)) hide)
     )
@@
   (symbol (lib_id "power:GND") (at 248.92 55.88 0) (unit 1)
     (in_bom yes) (on_board yes) (fields_autoplaced)
-    (property "Reference" "#PWR032" (id 0) (at 248.92 62.23 0)
+    (property "Reference" "#PWR033" (id 0) (at 248.92 62.23 0)
       (effects (font (size 1.27 1.27)) hide)
     )
@@
       (reference "#PWR030") (unit 1) (value "GND") (footprint "")
     )
+    (path "/22df3d09-cadc-45d9-88be-a191be084306"
+      (reference "#PWR031") (unit 1) (value "GND") (footprint "")
+    )
     (path "/48605c44-d3d1-4843-8bb5-ee84c23f92be"
-      (reference "#PWR031") (unit 1) (value "+BATT") (footprint "")
+      (reference "#PWR032") (unit 1) (value "+BATT") (footprint "")
     )
     (path "/f6fc2726-ba84-4c75-a80f-469493eaa4e1"
-      (reference "#PWR032") (unit 1) (value "GND") (footprint "")
+      (reference "#PWR033") (unit 1) (value "GND") (footprint "")
     )
     (path "/eb7973a1-d96b-484a-8470-c0ca08c82d7a"
-      (reference "#PWR033") (unit 1) (value "GND") (footprint "")
+      (reference "#PWR034") (unit 1) (value "GND") (footprint "")
     )
     (path "/96df7658-707a-48f0-825b-bd0b3ebf5148"
-      (reference "#PWR034") (unit 1) (value "GND") (footprint "")
+      (reference "#PWR035") (unit 1) (value "GND") (footprint "")
     )
     (path "/affe767e-505f-4c6f-9eab-d74f1858b254"
-      (reference "#PWR035") (unit 1) (value "GND") (footprint "")
+      (reference "#PWR036") (unit 1) (value "GND") (footprint "")
     )
     (path "/dee1721c-7498-4aa5-ba4d-8809f87db910"
@@
     )
     (path "/199564e9-96da-49ce-aee2-4093db89e0a3"
-      (reference "R3") (unit 1) (value "100K") (footprint "Resistor_SMD:R_0805_2012Metric")
+      (reference "R3") (unit 1) (value "100K") (footprint "Resistor_SMD:R_1206_3216Metric")
     )
     (path "/4ead0ca1-aaf2-482d-b51c-2ffe077e1536"
-      (reference "R4") (unit 1) (value "100K") (footprint "Resistor_SMD:R_0805_2012Metric")
+      (reference "R4") (unit 1) (value "100K") (footprint "Resistor_SMD:R_1206_3216Metric")
     )
     (path "/edbf3257-cd07-4b05-a56d-1984b019bc3d"
@@
     )
     (path "/59cd26eb-6e63-4857-a984-ee928ccec899"
-      (reference "R7") (unit 1) (value "100R") (footprint "Resistor_SMD:R_0805_2012Metric")
+      (reference "R7") (unit 1) (value "100R") (footprint "Resistor_SMD:R_1206_3216Metric")
     )
     (path "/e6d1af79-d7c7-41f9-85d8-9729ef258901"
-      (reference "R8") (unit 1) (value "10K") (footprint "Resistor_SMD:R_0805_2012Metric")
+      (reference "R8") (unit 1) (value "10K") (footprint "Resistor_SMD:R_1206_3216Metric")
     )
     (path "/b5cc64de-c33d-4294-8351-c594caa2bce6"
-      (reference "R9") (unit 1) (value "10K") (footprint "Resistor_SMD:R_0805_2012Metric")
+      (reference "R9") (unit 1) (value "22K") (footprint "Resistor_SMD:R_1206_3216Metric")
     )
     (path "/ea20ca82-5b13-40f2-8490-5e4e92c8de31"
-      (reference "R10") (unit 1) (value "10K") (footprint "Resistor_SMD:R_0805_2012Metric")
+      (reference "R10") (unit 1) (value "10K") (footprint "Resistor_SMD:R_1206_3216Metric")
+    )
+    (path "/44ac684e-df22-4ba9-b0ef-36d4bf4babc1"
+      (reference "R11") (unit 1) (value "33K") (footprint "Resistor_SMD:R_1206_3216Metric")
     )
     (path "/5b1d2768-c9d1-49e6-9cc7-584bddc858d7"
-      (reference "R11") (unit 1) (value "10K") (footprint "Resistor_SMD:R_0805_2012Metric")
+      (reference "R12") (unit 1) (value "10K") (footprint "Resistor_SMD:R_1206_3216Metric")
     )
     (path "/bb0c6fa2-b094-40f8-86ea-7ad2da51a06c"
