File: piridium-bus/Solar.kicad_sch (KiCad schematic)
At the start: 24 parts, among them J6 IN1, J7 IN2, U10 INA180A3, U9 LT3652EMSE

Commit message: route data lines, begin to route MPPT circuitry
Parts:
- renumbered C21 to C22, C22 to C23, C23 to C24, C24 to C25, C25 to C26
Changed lines of the file:
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@@
   (symbol (lib_id "Device:C") (at 199.39 66.04 90) (unit 1)
     (in_bom yes) (on_board yes)
-    (property "Reference" "C25" (id 0) (at 200.66 62.23 90)
+    (property "Reference" "C26" (id 0) (at 200.66 62.23 90)
       (effects (font (size 1.27 1.27)) (justify right))
     )
@@
   (symbol (lib_id "Device:C") (at 104.14 52.07 0) (unit 1)
     (in_bom yes) (on_board yes)
-    (property "Reference" "C22" (id 0) (at 107.061 50.9016 0)
+    (property "Reference" "C23" (id 0) (at 107.061 50.9016 0)
       (effects (font (size 1.27 1.27)) (justify left))
     )
@@
   (symbol (lib_id "Device:C") (at 66.04 73.66 0) (mirror y) (unit 1)
     (in_bom yes) (on_board yes)
-    (property "Reference" "C21" (id 0) (at 63.5 72.39 0)
+    (property "Reference" "C22" (id 0) (at 63.5 72.39 0)
       (effects (font (size 1.27 1.27)) (justify left))
     )
@@
   (symbol (lib_id "Device:C") (at 143.51 54.61 0) (unit 1)
     (in_bom yes) (on_board yes)
-    (property "Reference" "C23" (id 0) (at 143.51 52.07 0)
+    (property "Reference" "C24" (id 0) (at 143.51 52.07 0)
       (effects (font (size 1.27 1.27)) (justify left))
     )
@@
   (symbol (lib_id "Device:C") (at 161.29 67.31 0) (unit 1)
     (in_bom yes) (on_board yes)
-    (property "Reference" "C24" (id 0) (at 164.211 66.1416 0)
-      (effects (font (size 1.27 1.27)) (justify left))
-    )
+    (property "Reference" "C25" (id 0) (at 164.211 66.1416 0)
+      (effects (font (size 1.27 1.27)) (justify left))
+    )

Commit message: prototype timing circuit for LCL reset
Parts:
- renumbered C22 to C24, C23 to C25, C24 to C26, C25 to C27, C26 to C28, R25 to R34, R26 to R35, R27 to R36, R28 to R37, R29 to R38, R30 to R39, R31 to R40, U9 to U11, U10 to U12
Changed lines of the file:
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@@
   (symbol (lib_id "Device:R") (at 149.86 74.93 180) (unit 1)
     (in_bom yes) (on_board yes)
-    (property "Reference" "R29" (id 0) (at 151.13 74.93 0)
+    (property "Reference" "R38" (id 0) (at 151.13 74.93 0)
       (effects (font (size 1.27 1.27)) (justify right))
     )
@@
   (symbol (lib_id "Device:R") (at 72.39 73.66 0) (unit 1)
     (in_bom yes) (on_board yes)
-    (property "Reference" "R26" (id 0) (at 73.66 73.66 0)
+    (property "Reference" "R35" (id 0) (at 73.66 73.66 0)
       (effects (font (size 1.27 1.27)) (justify left))
     )
@@
   (symbol (lib_id "Device:C") (at 199.39 66.04 90) (unit 1)
     (in_bom yes) (on_board yes)
-    (property "Reference" "C26" (id 0) (at 200.66 62.23 90)
+    (property "Reference" "C28" (id 0) (at 200.66 62.23 90)
       (effects (font (size 1.27 1.27)) (justify right))
     )
@@
   (symbol (lib_id "power:GND") (at 151.13 45.72 0) (unit 1)
     (in_bom yes) (on_board yes)
-    (property "Reference" "#PWR050" (id 0) (at 151.13 52.07 0)
+    (property "Reference" "#PWR057" (id 0) (at 151.13 52.07 0)
       (effects (font (size 1.27 1.27)) hide)
     )
@@
   (symbol (lib_id "Device:R") (at 166.37 60.96 270) (unit 1)
     (in_bom yes) (on_board yes)
-    (property "Reference" "R30" (id 0) (at 170.18 58.42 90))
+    (property "Reference" "R39" (id 0) (at 170.18 58.42 90))
     (property "Value" "50m" (id 1) (at 166.37 60.96 90))
     (property "Footprint" "Resistor_SMD:R_1206_3216Metric" (id 2) (at 166.37 59.182 90)
@@
   (symbol (lib_id "power:GND") (at 36.83 59.69 0) (unit 1)
     (in_bom yes) (on_board yes) (fields_autoplaced)
-    (property "Reference" "#PWR048" (id 0) (at 36.83 66.04 0)
+    (property "Reference" "#PWR055" (id 0) (at 36.83 66.04 0)
       (effects (font (size 1.27 1.27)) hide)
     )
@@
   (symbol (lib_id "Device:R") (at 144.78 71.12 270) (unit 1)
     (in_bom yes) (on_board yes)
-    (property "Reference" "R27" (id 0) (at 144.78 68.58 90))
+    (property "Reference" "R36" (id 0) (at 144.78 68.58 90))
     (property "Value" "191K" (id 1) (at 144.78 71.12 90))
     (property "Footprint" "Resistor_SMD:R_0805_2012Metric" (id 2) (at 144.78 69.342 90)
@@
   (symbol (lib_id "Device:C") (at 104.14 52.07 0) (unit 1)
     (in_bom yes) (on_board yes)
-    (property "Reference" "C23" (id 0) (at 107.061 50.9016 0)
+    (property "Reference" "C25" (id 0) (at 107.061 50.9016 0)
       (effects (font (size 1.27 1.27)) (justify left))
     )
@@
   (symbol (lib_id "Amplifier_Current:INA138") (at 198.12 73.66 0) (unit 1)
     (in_bom yes) (on_board yes)
-    (property "Reference" "U10" (id 0) (at 206.8576 72.4916 0)
+    (property "Reference" "U12" (id 0) (at 206.8576 72.4916 0)
       (effects (font (size 1.27 1.27)) (justify left))
     )
@@
   (symbol (lib_id "Device:R") (at 149.86 67.31 180) (unit 1)
     (in_bom yes) (on_board yes)
-    (property "Reference" "R28" (id 0) (at 151.13 67.31 0)
+    (property "Reference" "R37" (id 0) (at 151.13 67.31 0)
       (effects (font (size 1.27 1.27)) (justify right))
     )
@@
   (symbol (lib_id "Device:R") (at 72.39 53.34 0) (unit 1)
     (in_bom yes) (on_board yes)
-    (property "Reference" "R25" (id 0) (at 73.66 53.34 0)
+    (property "Reference" "R34" (id 0) (at 73.66 53.34 0)
       (effects (font (size 1.27 1.27)) (justify left))
     )
@@
   (symbol (lib_id "power:GND") (at 36.83 43.18 0) (unit 1)
     (in_bom yes) (on_board yes) (fields_autoplaced)
-    (property "Reference" "#PWR047" (id 0) (at 36.83 49.53 0)
+    (property "Reference" "#PWR054" (id 0) (at 36.83 49.53 0)
       (effects (font (size 1.27 1.27)) hide)
     )
@@
   (symbol (lib_id "power:GND") (at 76.2 78.74 0) (unit 1)
     (in_bom yes) (on_board yes)
-    (property "Reference" "#PWR049" (id 0) (at 76.2 85.09 0)
+    (property "Reference" "#PWR056" (id 0) (at 76.2 85.09 0)
       (effects (font (size 1.27 1.27)) hide)
     )
@@
   (symbol (lib_id "Device:C") (at 66.04 73.66 0) (mirror y) (unit 1)
     (in_bom yes) (on_board yes)
-    (property "Reference" "C22" (id 0) (at 63.5 72.39 0)
+    (property "Reference" "C24" (id 0) (at 63.5 72.39 0)
       (effects (font (size 1.27 1.27)) (justify left))
     )
@@
   (symbol (lib_id "Device:R") (at 184.15 60.96 270) (unit 1)
     (in_bom yes) (on_board yes)
-    (property "Reference" "R31" (id 0) (at 184.15 58.42 90))
+    (property "Reference" "R40" (id 0) (at 184.15 58.42 90))
     (property "Value" "4m" (id 1) (at 184.15 60.96 90))
     (property "Footprint" "Resistor_SMD:R_1206_3216Metric" (id 2) (at 184.15 59.182 90)
@@
   (symbol (lib_id "power:+3.3V") (at 195.58 66.04 0) (unit 1)
     (in_bom yes) (on_board yes)
-    (property "Reference" "#PWR051" (id 0) (at 195.58 69.85 0)
+    (property "Reference" "#PWR058" (id 0) (at 195.58 69.85 0)
       (effects (font (size 1.27 1.27)) hide)
     )
@@
   (symbol (lib_id "power:GND") (at 195.58 81.28 0) (unit 1)
     (in_bom yes) (on_board yes)
-    (property "Reference" "#PWR052" (id 0) (at 195.58 87.63 0)
+    (property "Reference" "#PWR059" (id 0) (at 195.58 87.63 0)
       (effects (font (size 1.27 1.27)) hide)
     )
@@
   (symbol (lib_id "Device:C") (at 143.51 54.61 0) (unit 1)
     (in_bom yes) (on_board yes)
-    (property "Reference" "C24" (id 0) (at 143.51 52.07 0)
+    (property "Reference" "C26" (id 0) (at 143.51 52.07 0)
       (effects (font (size 1.27 1.27)) (justify left))
     )
@@
   (symbol (lib_id "Battery_Management:LT3652EMSE") (at 127 60.96 0) (unit 1)
     (in_bom yes) (on_board yes)
-    (property "Reference" "U9" (id 0) (at 127 43.6626 0))
+    (property "Reference" "U11" (id 0) (at 127 43.6626 0))
     (property "Value" "LT3652EMSE" (id 1) (at 127 45.974 0))
     (property "Footprint" "Package_SO:MSOP-12-1EP_3x4mm_P0.65mm_EP1.65x2.85mm" (id 2) (at 127 76.2 0)
@@
   (symbol (lib_id "power:GND") (at 203.2 66.04 0) (unit 1)
     (in_bom yes) (on_board yes)
-    (property "Reference" "#PWR053" (id 0) (at 203.2 72.39 0)
+    (property "Reference" "#PWR060" (id 0) (at 203.2 72.39 0)
       (effects (font (size 1.27 1.27)) hide)
     )
@@
   (symbol (lib_id "Device:C") (at 161.29 67.31 0) (unit 1)
     (in_bom yes) (on_board yes)
-    (property "Reference" "C25" (id 0) (at 164.211 66.1416 0)
-      (effects (font (size 1.27 1.27)) (justify left))
-    )
+    (property "Reference" "C27" (id 0) (at 164.211 66.1416 0)
+      (effects (font (size 1.27 1.27)) (justify left))
+    )

Commit message: battery sch finish
Parts:
- renumbered C24 to C22, C25 to C23, C26 to C24, C27 to C25, C28 to C26, R34 to R29, R35 to R30, R36 to R31, R37 to R32, R38 to R33, R39 to R34, R40 to R35, U12 to U10, U11 to U9
Changed lines of the file:
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@@
   (symbol (lib_id "Device:R") (at 149.86 74.93 180) (unit 1)
     (in_bom yes) (on_board yes)
-    (property "Reference" "R38" (id 0) (at 151.13 74.93 0)
+    (property "Reference" "R33" (id 0) (at 151.13 74.93 0)
       (effects (font (size 1.27 1.27)) (justify right))
     )
@@
   (symbol (lib_id "Device:R") (at 72.39 73.66 0) (unit 1)
     (in_bom yes) (on_board yes)
-    (property "Reference" "R35" (id 0) (at 73.66 73.66 0)
+    (property "Reference" "R30" (id 0) (at 73.66 73.66 0)
       (effects (font (size 1.27 1.27)) (justify left))
     )
@@
   (symbol (lib_id "Device:C") (at 199.39 66.04 90) (unit 1)
     (in_bom yes) (on_board yes)
-    (property "Reference" "C28" (id 0) (at 200.66 62.23 90)
+    (property "Reference" "C26" (id 0) (at 200.66 62.23 90)
       (effects (font (size 1.27 1.27)) (justify right))
     )
@@
   (symbol (lib_id "power:GND") (at 151.13 45.72 0) (unit 1)
     (in_bom yes) (on_board yes)
-    (property "Reference" "#PWR057" (id 0) (at 151.13 52.07 0)
+    (property "Reference" "#PWR053" (id 0) (at 151.13 52.07 0)
       (effects (font (size 1.27 1.27)) hide)
     )
@@
   (symbol (lib_id "Device:R") (at 166.37 60.96 270) (unit 1)
     (in_bom yes) (on_board yes)
-    (property "Reference" "R39" (id 0) (at 170.18 58.42 90))
+    (property "Reference" "R34" (id 0) (at 170.18 58.42 90))
     (property "Value" "50m" (id 1) (at 166.37 60.96 90))
     (property "Footprint" "Resistor_SMD:R_1206_3216Metric" (id 2) (at 166.37 59.182 90)
@@
   (symbol (lib_id "power:GND") (at 36.83 59.69 0) (unit 1)
     (in_bom yes) (on_board yes) (fields_autoplaced)
-    (property "Reference" "#PWR055" (id 0) (at 36.83 66.04 0)
+    (property "Reference" "#PWR051" (id 0) (at 36.83 66.04 0)
       (effects (font (size 1.27 1.27)) hide)
     )
@@
   (symbol (lib_id "Device:R") (at 144.78 71.12 270) (unit 1)
     (in_bom yes) (on_board yes)
-    (property "Reference" "R36" (id 0) (at 144.78 68.58 90))
+    (property "Reference" "R31" (id 0) (at 144.78 68.58 90))
     (property "Value" "191K" (id 1) (at 144.78 71.12 90))
     (property "Footprint" "Resistor_SMD:R_0805_2012Metric" (id 2) (at 144.78 69.342 90)
@@
   (symbol (lib_id "Device:C") (at 104.14 52.07 0) (unit 1)
     (in_bom yes) (on_board yes)
-    (property "Reference" "C25" (id 0) (at 107.061 50.9016 0)
+    (property "Reference" "C23" (id 0) (at 107.061 50.9016 0)
       (effects (font (size 1.27 1.27)) (justify left))
     )
@@
   (symbol (lib_id "Amplifier_Current:INA138") (at 198.12 73.66 0) (unit 1)
     (in_bom yes) (on_board yes)
-    (property "Reference" "U12" (id 0) (at 206.8576 72.4916 0)
+    (property "Reference" "U10" (id 0) (at 206.8576 72.4916 0)
       (effects (font (size 1.27 1.27)) (justify left))
     )
@@
   (symbol (lib_id "Device:R") (at 149.86 67.31 180) (unit 1)
     (in_bom yes) (on_board yes)
-    (property "Reference" "R37" (id 0) (at 151.13 67.31 0)
+    (property "Reference" "R32" (id 0) (at 151.13 67.31 0)
       (effects (font (size 1.27 1.27)) (justify right))
     )
@@
   (symbol (lib_id "Device:R") (at 72.39 53.34 0) (unit 1)
     (in_bom yes) (on_board yes)
-    (property "Reference" "R34" (id 0) (at 73.66 53.34 0)
+    (property "Reference" "R29" (id 0) (at 73.66 53.34 0)
       (effects (font (size 1.27 1.27)) (justify left))
     )
@@
   (symbol (lib_id "power:GND") (at 36.83 43.18 0) (unit 1)
     (in_bom yes) (on_board yes) (fields_autoplaced)
-    (property "Reference" "#PWR054" (id 0) (at 36.83 49.53 0)
+    (property "Reference" "#PWR050" (id 0) (at 36.83 49.53 0)
       (effects (font (size 1.27 1.27)) hide)
     )
@@
   (symbol (lib_id "power:GND") (at 76.2 78.74 0) (unit 1)
     (in_bom yes) (on_board yes)
-    (property "Reference" "#PWR056" (id 0) (at 76.2 85.09 0)
+    (property "Reference" "#PWR052" (id 0) (at 76.2 85.09 0)
       (effects (font (size 1.27 1.27)) hide)
     )
@@
   (symbol (lib_id "Device:C") (at 66.04 73.66 0) (mirror y) (unit 1)
     (in_bom yes) (on_board yes)
-    (property "Reference" "C24" (id 0) (at 63.5 72.39 0)
+    (property "Reference" "C22" (id 0) (at 63.5 72.39 0)
       (effects (font (size 1.27 1.27)) (justify left))
     )
@@
   (symbol (lib_id "Device:R") (at 184.15 60.96 270) (unit 1)
     (in_bom yes) (on_board yes)
-    (property "Reference" "R40" (id 0) (at 184.15 58.42 90))
+    (property "Reference" "R35" (id 0) (at 184.15 58.42 90))
     (property "Value" "4m" (id 1) (at 184.15 60.96 90))
     (property "Footprint" "Resistor_SMD:R_1206_3216Metric" (id 2) (at 184.15 59.182 90)
@@
   (symbol (lib_id "power:+3.3V") (at 195.58 66.04 0) (unit 1)
     (in_bom yes) (on_board yes)
-    (property "Reference" "#PWR058" (id 0) (at 195.58 69.85 0)
+    (property "Reference" "#PWR054" (id 0) (at 195.58 69.85 0)
       (effects (font (size 1.27 1.27)) hide)
     )
@@
   (symbol (lib_id "power:GND") (at 195.58 81.28 0) (unit 1)
     (in_bom yes) (on_board yes)
-    (property "Reference" "#PWR059" (id 0) (at 195.58 87.63 0)
+    (property "Reference" "#PWR055" (id 0) (at 195.58 87.63 0)
       (effects (font (size 1.27 1.27)) hide)
     )
@@
   (symbol (lib_id "Device:C") (at 143.51 54.61 0) (unit 1)
     (in_bom yes) (on_board yes)
-    (property "Reference" "C26" (id 0) (at 143.51 52.07 0)
+    (property "Reference" "C24" (id 0) (at 143.51 52.07 0)
       (effects (font (size 1.27 1.27)) (justify left))
     )
@@
   (symbol (lib_id "Battery_Management:LT3652EMSE") (at 127 60.96 0) (unit 1)
     (in_bom yes) (on_board yes)
-    (property "Reference" "U11" (id 0) (at 127 43.6626 0))
+    (property "Reference" "U9" (id 0) (at 127 43.6626 0))
     (property "Value" "LT3652EMSE" (id 1) (at 127 45.974 0))
     (property "Footprint" "Package_SO:MSOP-12-1EP_3x4mm_P0.65mm_EP1.65x2.85mm" (id 2) (at 127 76.2 0)
@@
   (symbol (lib_id "power:GND") (at 203.2 66.04 0) (unit 1)
     (in_bom yes) (on_board yes)
-    (property "Reference" "#PWR060" (id 0) (at 203.2 72.39 0)
+    (property "Reference" "#PWR056" (id 0) (at 203.2 72.39 0)
       (effects (font (size 1.27 1.27)) hide)
     )
@@
   (symbol (lib_id "Device:C") (at 161.29 67.31 0) (unit 1)
     (in_bom yes) (on_board yes)
-    (property "Reference" "C27" (id 0) (at 164.211 66.1416 0)
-      (effects (font (size 1.27 1.27)) (justify left))
-    )
+    (property "Reference" "C25" (id 0) (at 164.211 66.1416 0)
+      (effects (font (size 1.27 1.27)) (justify left))
+    )

Commit message: mcp3208 constant reference
Parts:
- renumbered U9 to U10, U10 to U11
Changed lines of the file:
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@@
   (symbol (lib_id "power:GND") (at 151.13 45.72 0) (unit 1)
     (in_bom yes) (on_board yes)
-    (property "Reference" "#PWR053" (id 0) (at 151.13 52.07 0)
+    (property "Reference" "#PWR055" (id 0) (at 151.13 52.07 0)
       (effects (font (size 1.27 1.27)) hide)
     )
@@
   (symbol (lib_id "power:GND") (at 36.83 59.69 0) (unit 1)
     (in_bom yes) (on_board yes) (fields_autoplaced)
-    (property "Reference" "#PWR051" (id 0) (at 36.83 66.04 0)
+    (property "Reference" "#PWR053" (id 0) (at 36.83 66.04 0)
       (effects (font (size 1.27 1.27)) hide)
     )
@@
   (symbol (lib_id "Amplifier_Current:INA138") (at 198.12 73.66 0) (unit 1)
     (in_bom yes) (on_board yes)
-    (property "Reference" "U10" (id 0) (at 206.8576 72.4916 0)
+    (property "Reference" "U11" (id 0) (at 206.8576 72.4916 0)
       (effects (font (size 1.27 1.27)) (justify left))
     )
@@
   (symbol (lib_id "power:GND") (at 36.83 43.18 0) (unit 1)
     (in_bom yes) (on_board yes) (fields_autoplaced)
-    (property "Reference" "#PWR050" (id 0) (at 36.83 49.53 0)
+    (property "Reference" "#PWR052" (id 0) (at 36.83 49.53 0)
       (effects (font (size 1.27 1.27)) hide)
     )
@@
   (symbol (lib_id "power:GND") (at 76.2 78.74 0) (unit 1)
     (in_bom yes) (on_board yes)
-    (property "Reference" "#PWR052" (id 0) (at 76.2 85.09 0)
+    (property "Reference" "#PWR054" (id 0) (at 76.2 85.09 0)
       (effects (font (size 1.27 1.27)) hide)
     )
@@
   (symbol (lib_id "power:+3.3V") (at 195.58 66.04 0) (unit 1)
     (in_bom yes) (on_board yes)
-    (property "Reference" "#PWR054" (id 0) (at 195.58 69.85 0)
+    (property "Reference" "#PWR056" (id 0) (at 195.58 69.85 0)
       (effects (font (size 1.27 1.27)) hide)
     )
@@
   (symbol (lib_id "power:GND") (at 195.58 81.28 0) (unit 1)
     (in_bom yes) (on_board yes)
-    (property "Reference" "#PWR055" (id 0) (at 195.58 87.63 0)
+    (property "Reference" "#PWR057" (id 0) (at 195.58 87.63 0)
       (effects (font (size 1.27 1.27)) hide)
     )
@@
   (symbol (lib_id "Battery_Management:LT3652EMSE") (at 127 60.96 0) (unit 1)
     (in_bom yes) (on_board yes)
-    (property "Reference" "U9" (id 0) (at 127 43.6626 0))
+    (property "Reference" "U10" (id 0) (at 127 43.6626 0))
     (property "Value" "LT3652EMSE" (id 1) (at 127 45.974 0))
     (property "Footprint" "Package_SO:MSOP-12-1EP_3x4mm_P0.65mm_EP1.65x2.85mm" (id 2) (at 127 76.2 0)
@@
   (symbol (lib_id "power:GND") (at 203.2 66.04 0) (unit 1)
     (in_bom yes) (on_board yes)
-    (property "Reference" "#PWR056" (id 0) (at 203.2 72.39 0)
-      (effects (font (size 1.27 1.27)) hide)
-    )
+    (property "Reference" "#PWR058" (id 0) (at 203.2 72.39 0)
+      (effects (font (size 1.27 1.27)) hide)
+    )

Commit message: pull down on/off instead of up
Parts:
- renumbered R29 to R28, R30 to R29, R31 to R30, R32 to R31, R33 to R32, R34 to R33, R35 to R34
Changed lines of the file:
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@@
   (symbol (lib_id "Device:R") (at 149.86 74.93 180) (unit 1)
     (in_bom yes) (on_board yes)
-    (property "Reference" "R33" (id 0) (at 151.13 74.93 0)
+    (property "Reference" "R32" (id 0) (at 151.13 74.93 0)
       (effects (font (size 1.27 1.27)) (justify right))
     )
@@
   (symbol (lib_id "Device:R") (at 72.39 73.66 0) (unit 1)
     (in_bom yes) (on_board yes)
-    (property "Reference" "R30" (id 0) (at 73.66 73.66 0)
+    (property "Reference" "R29" (id 0) (at 73.66 73.66 0)
       (effects (font (size 1.27 1.27)) (justify left))
     )
@@
   (symbol (lib_id "power:GND") (at 151.13 45.72 0) (unit 1)
     (in_bom yes) (on_board yes)
-    (property "Reference" "#PWR055" (id 0) (at 151.13 52.07 0)
+    (property "Reference" "#PWR054" (id 0) (at 151.13 52.07 0)
       (effects (font (size 1.27 1.27)) hide)
     )
@@
   (symbol (lib_id "Device:R") (at 166.37 60.96 270) (unit 1)
     (in_bom yes) (on_board yes)
-    (property "Reference" "R34" (id 0) (at 170.18 58.42 90))
+    (property "Reference" "R33" (id 0) (at 170.18 58.42 90))
     (property "Value" "50m" (id 1) (at 166.37 60.96 90))
     (property "Footprint" "Resistor_SMD:R_1206_3216Metric" (id 2) (at 166.37 59.182 90)
@@
   (symbol (lib_id "power:GND") (at 36.83 59.69 0) (unit 1)
     (in_bom yes) (on_board yes) (fields_autoplaced)
-    (property "Reference" "#PWR053" (id 0) (at 36.83 66.04 0)
+    (property "Reference" "#PWR052" (id 0) (at 36.83 66.04 0)
       (effects (font (size 1.27 1.27)) hide)
     )
@@
   (symbol (lib_id "Device:R") (at 144.78 71.12 270) (unit 1)
     (in_bom yes) (on_board yes)
-    (property "Reference" "R31" (id 0) (at 144.78 68.58 90))
+    (property "Reference" "R30" (id 0) (at 144.78 68.58 90))
     (property "Value" "191K" (id 1) (at 144.78 71.12 90))
     (property "Footprint" "Resistor_SMD:R_0805_2012Metric" (id 2) (at 144.78 69.342 90)
@@
   (symbol (lib_id "Device:R") (at 149.86 67.31 180) (unit 1)
     (in_bom yes) (on_board yes)
-    (property "Reference" "R32" (id 0) (at 151.13 67.31 0)
+    (property "Reference" "R31" (id 0) (at 151.13 67.31 0)
       (effects (font (size 1.27 1.27)) (justify right))
     )
@@
   (symbol (lib_id "Device:R") (at 72.39 53.34 0) (unit 1)
     (in_bom yes) (on_board yes)
-    (property "Reference" "R29" (id 0) (at 73.66 53.34 0)
+    (property "Reference" "R28" (id 0) (at 73.66 53.34 0)
       (effects (font (size 1.27 1.27)) (justify left))
     )
@@
   (symbol (lib_id "power:GND") (at 36.83 43.18 0) (unit 1)
     (in_bom yes) (on_board yes) (fields_autoplaced)
-    (property "Reference" "#PWR052" (id 0) (at 36.83 49.53 0)
+    (property "Reference" "#PWR051" (id 0) (at 36.83 49.53 0)
       (effects (font (size 1.27 1.27)) hide)
     )
@@
   (symbol (lib_id "power:GND") (at 76.2 78.74 0) (unit 1)
     (in_bom yes) (on_board yes)
-    (property "Reference" "#PWR054" (id 0) (at 76.2 85.09 0)
+    (property "Reference" "#PWR053" (id 0) (at 76.2 85.09 0)
       (effects (font (size 1.27 1.27)) hide)
     )
@@
   (symbol (lib_id "Device:R") (at 184.15 60.96 270) (unit 1)
     (in_bom yes) (on_board yes)
-    (property "Reference" "R35" (id 0) (at 184.15 58.42 90))
+    (property "Reference" "R34" (id 0) (at 184.15 58.42 90))
     (property "Value" "4m" (id 1) (at 184.15 60.96 90))
     (property "Footprint" "Resistor_SMD:R_1206_3216Metric" (id 2) (at 184.15 59.182 90)
@@
   (symbol (lib_id "power:+3.3V") (at 195.58 66.04 0) (unit 1)
     (in_bom yes) (on_board yes)
-    (property "Reference" "#PWR056" (id 0) (at 195.58 69.85 0)
+    (property "Reference" "#PWR055" (id 0) (at 195.58 69.85 0)
       (effects (font (size 1.27 1.27)) hide)
     )
@@
   (symbol (lib_id "power:GND") (at 195.58 81.28 0) (unit 1)
     (in_bom yes) (on_board yes)
-    (property "Reference" "#PWR057" (id 0) (at 195.58 87.63 0)
+    (property "Reference" "#PWR056" (id 0) (at 195.58 87.63 0)
       (effects (font (size 1.27 1.27)) hide)
     )
@@
   (symbol (lib_id "power:GND") (at 203.2 66.04 0) (unit 1)
     (in_bom yes) (on_board yes)
-    (property "Reference" "#PWR058" (id 0) (at 203.2 72.39 0)
-      (effects (font (size 1.27 1.27)) hide)
-    )
+    (property "Reference" "#PWR057" (id 0) (at 203.2 72.39 0)
+      (effects (font (size 1.27 1.27)) hide)
+    )
