File: piridium-eps/piridium-eps.kicad_pcb (KiCad board)
At the start: 4 copper layers, 90.2 x 95.9 mm, 30 parts, among them J1 EPS, Q1 Si4186DY, Q2 Si4186DY, U1 BQ29209, U2 R5460N212AF

Commit message: license
Parts:
- BT2: footprint Battery:BatteryHolder_Keystone_1042_1x18650 -> piridium-eps:Keystone_1042_1x18650_Shortpad
- BT3: footprint Battery:BatteryHolder_Keystone_1042_1x18650 -> piridium-eps:Keystone_1042_1x18650_Shortpad2
- moved R5 133.9 mm to (163.4, 99.0), turned to 180 degrees
- moved R6 130.0 mm to (160.1, 94.8), turned to -90 degrees
- moved R2 128.6 mm to (174.6, 95.6), turned to 180 degrees
- moved R4 125.4 mm to (167.2, 101.4)
- moved R3 122.9 mm to (167.2, 99.1)
- moved R7 121.1 mm to (163.4, 102.6)
- moved C6 117.3 mm to (159.3, 97.7), turned to 180 degrees
- moved C2 110.4 mm to (171.5, 96.6), turned to -90 degrees
- moved R1 107.0 mm to (179.6, 96.6), turned to -90 degrees
- moved C3 100.9 mm to (171.5, 100.1), turned to -90 degrees
- moved C7 96.0 mm to (161.4, 105.3), turned to 90 degrees
- moved C4 92.1 mm to (175.1, 103.7)
- moved U2 90.5 mm to (159.9, 101.5), turned to 90 degrees
- moved C5 89.9 mm to (163.4, 105.3), turned to -90 degrees
- moved C1 85.2 mm to (179.6, 100.4), turned to -90 degrees
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Routing:
- net Net-(BT1-Pad2): track 0.00 -> 66.3 mm
- net -BATT: track 0.00 -> 47.5 mm, vias 0 -> 5
- net +BATT: track 0.00 -> 44.0 mm, vias 0 -> 3
- net Net-(Q1-Pad5): track 0.00 -> 10.7 mm
- net Net-(Q2-Pad4): track 0.00 -> 10.1 mm
- net GND: track 0.00 -> 9.17 mm
- net Net-(C2-Pad2): track 0.00 -> 7.66 mm
- net Net-(C5-Pad1): track 0.00 -> 7.38 mm
- net Net-(Q1-Pad4): track 0.00 -> 6.18 mm
- net Net-(C6-Pad1): track 0.00 -> 4.91 mm
- net Net-(C1-Pad1): track 0.00 -> 4.42 mm
- net Net-(C7-Pad2): track 0.00 -> 3.70 mm
- net Net-(C3-Pad2): track 0.00 -> 3.54 mm
- net Net-(C2-Pad1): track 0.00 -> 2.16 mm

Commit message: finish battery
Parts:
- removed F1: 7A, Resistor_SMD:R_1206_3216Metric
- added R8: 20m, Resistor_SMD:R_2512_6332Metric, F.Cu at (173.7, 108.5)
- BT6: footprint Battery:BatteryHolder_Keystone_1042_1x18650 -> piridium-eps:Keystone_1042_1x18650_Shortpad3
- moved BT5 8.13 mm to (136.4, 98.8)
- moved BT6 8.13 mm to (115.1, 98.8)
Connections:
- J1 pad 1: Net-(F1-Pad2) -> +BATT
- Q2 pad 1: GND -> Net-(Q2-Pad1)
- Q2 pad 2: GND -> Net-(Q2-Pad1)
- Q2 pad 3: GND -> Net-(Q2-Pad1)
Routing:
- net +BATT: track 44.0 -> 193.7 mm
- net Net-(BT1-Pad2): track 66.3 -> 181.0 mm, vias 0 -> 7
- net -BATT: track 47.5 -> 133.2 mm, vias 5 -> 6
- net GND: track 9.17 -> 15.8 mm, vias 0 -> 1
- net Net-(Q2-Pad1): track 0.00 -> 4.66 mm
- net Net-(C4-Pad1): track 0.00 -> 2.62 mm
- net Net-(C3-Pad2): track 3.54 -> 6.11 mm
- added copper zone on B.Cu, net GND
- added copper zone on F.Cu, net GND
Other:
- board text added: "+"
- board text added: "-"
- board text added: "BATT+"
- board text added: "BATT-"
- board text added: "Board Comments"
- board text added: "Piridium Battery Board github.com/Alan-JH/piridium-bus v1"

Commit message: switch battery to 2 layer
Other:
- copper layers 4 -> 2
Changed lines of the file:
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@@
 (kicad_pcb (version 20211014) (generator pcbnew)
   (general
-    (thickness 1.56)
+    (thickness 0.19)
   )
   (paper "A4")
   (layers
     (0 "F.Cu" signal)
-    (1 "In1.Cu" signal)
-    (2 "In2.Cu" signal)
     (31 "B.Cu" signal)
     (32 "B.Adhes" user "B.Adhesive")
@@
       (layer "F.Cu" (type "copper") (thickness 0.035))
       (layer "dielectric 1" (type "core") (thickness 0.1) (material "FR4") (epsilon_r 4.5) (loss_tangent 0.02))
-      (layer "In1.Cu" (type "copper") (thickness 0.035))
-      (layer "dielectric 2" (type "prepreg") (thickness 1.2) (material "FR4") (epsilon_r 4.5) (loss_tangent 0.02))
-      (layer "In2.Cu" (type "copper") (thickness 0.035))
-      (layer "dielectric 3" (type "core") (thickness 0.1) (material "FR4") (epsilon_r 4.5) (loss_tangent 0.02))
       (layer "B.Cu" (type "copper") (thickness 0.035))
       (layer "B.Mask" (type "Bottom Solder Mask") (thickness 0.01))
